File: Hardware/InkTime_Schematic.sch (EAGLE design)
At the start: 57 parts, among them IC1 BQ25180YBGR, IC3 BMA423_BMA423, IC9 RT6160AWSC_RT6160AWSC, J1 TC2030-IDC_TC2030-IDC, X1 32MHz, X2 32.768kHz

Commit message: Finished schematic implementation
Parts:
- removed R1: CPF0201D7K68C1_CPF0201D7K68C1, InkTime_v5:CPF0201D7K68C1_CPF0201D7K68C1
- added C1-EP-DR: 10uF, InkTime_v5:NORDIC_NRF_3_CAPACITOR_0402_L
- added C2-EP-DR1: 4.7uF/25V, InkTime_v5:NORDIC_NRF_3_CAPACITOR_0402_L
- added C27, C42: 0.1uF, InkTime_v5:NORDIC_NRF_3_CAPACITOR_0201_L
- added C29, C30, C31: 1uF, InkTime_v5:NORDIC_NRF_3_CAPACITOR_0402_L
- added C32: 1uF, InkTime_v5:GRM011R60J152KE01L_2_GRM011R60J152KE01L
- added C34: 0.1uF, InkTime_v5:GRM011R60J152KE01L_2_GRM011R60J152KE01L
- added C43: 4.7uF, InkTime_v5:NORDIC_NRF_3_CAPACITOR_0402_L
- added D2, D4, D5: MBR0530, InkTime_v5:ESP32_C6_LIBRARY_5_MBR0530
- added D3: USBLC6-2SC6Y, InkTime_v5:ESP32_C6_LIBRARY_3_USBLC6-2SC6Y
- added EPD_C1, EPD_C10, EPD_C11, EPD_C12, EPD_C2, EPD_C6, EPD_C7, EPD_C8, EPD_C9: 1uF/50V, InkTime_v5:NORDIC_NRF_3_CAPACITOR_0402_L
- added EPD_C5: 0.1uF/50V, InkTime_v5:NORDIC_NRF_3_CAPACITOR_0201_L
- added IC2: DRV2605YZFR, InkTime_v5:DRV2605YZFR_DRV2605YZFR
- added J2: TC2030-IDC, InkTime_v5:TC2030-IDC_TC2030-IDC
- added J4: KH-TYPE-C-16P, InkTime_v5:KH-TYPE-C-16P_KH-TYPE-C-16P
- added L5: 68uH, InkTime_v5:ESP32_C6_LIBRARY_2_744043680IND_4828-WE-TPC_WRE
- added Q1: 20V/4.2A/52mΩ/1.4W, InkTime_v5:ESP32_C6_LIBRARY_4_ESP32_WROVER_SPARKFUN-DISCRETESEMI_MOSFET_PCH-DMG2305UX-7
- added Q3: SI1308EDL-T1-GE3, InkTime_v5:ESP32_C6_LIBRARY_6_SI1308EDL-T1-GE3
- added R1_EP_DR: 0.47, InkTime_v5:CPF0201D7K68C1_CPF0201D7K68C1
- added R1_USB, R2_USB: 5K1, InkTime_v5:ERA-1AEB3401C_CPF0201D7K68C1
- added R2_EP_DR, R_PWR_EPD: 10K, InkTime_v5:CPF0201D7K68C1_CPF0201D7K68C1
- added R4: CPF0201D7K68C1_CPF0201D7K68C1, InkTime_v5:CPF0201D7K68C1_CPF0201D7K68C1
- added R5, R7, R8: 10k, InkTime_v5:CPF0201D7K68C1_CPF0201D7K68C1
- added R_TYPE_SEL: 2.2, InkTime_v5:CPF0201D7K68C1_CPF0201D7K68C1
- added SJ1: (no value), InkTime_v5:ESP32_C6_LIBRARY_7_JUMPER_SJ
- added SW_DN, SW_UP: 2025-10-22_07-23-44_LIBRARY_EVP-AKE31ASW_EVP-AKE31A_PAN, InkTime_v5:2025-10-22_07-23-44_LIBRARY_EVP-AKE31ASW_EVP-AKE31A_PAN
- added SW_ENT: SW_ENT, InkTime_v5:2025-10-22_07-23-44_LIBRARY_EVP-AKE31ASW_EVP-AKE31A_PAN
- added TP_BAT_GND, TP_ON, TP_OP, TP_VBAT: HECTOR_WATCH_1_TPTP20R, InkTime_v5:HECTOR_WATCH_1_TPTP20R
- added U3: MAX17048G+T10, InkTime_v5:ESP32_C6_LIBRARY_MAX17048G+T10
- C23: device InkTime_v5:GRM011R60J152KE01L_2_GRM011R60J152KE01L -> InkTime_v5:NORDIC_NRF_3_CAPACITOR_0201_L
- J1: value TC2030-IDC_TC2030-IDC -> 503480-2400; device InkTime_v5:TC2030-IDC_TC2030-IDC -> InkTime_v5:503480-2400_503480-2400
Connections:
- removed net N$20 (its old number): R1.2
- new net 3V3/1.7D: C34.2, IC2.VDD, Q1.S, R5.2, R7.2, R8.2, R_PWR_EPD.2
- new net ALERT/1.6C: U3.!ALERT
- new net D+/1.5D: D3.I/O2_2
- new net D-/1.5D: D3.I/O1_2
- new net DN: D3.I/O1_1, J4.DN1, J4.DN2
- new net DP: D3.I/O2_1, J4.DP1, J4.DP2
- new net EPD_3V3: C1-EP-DR.1, EPD_C5.2, J1.15, J1.16, L5.2, Q1.D
- new net EPD_BUSY/1.5D: J1.9
- new net EPD_CS/1.4C: J1.12
- new net EPD_DC/1.5D: J1.11
- new net EPD_RST/1.5D: J1.10
- new net GDR: J1.2, Q3.G, R2_EP_DR.2
- new net GND1: C2-EP-DR1.2, D5.A, L5.1, Q3.D
- new net HAPTIC_EN/1.4A: IC2.EN
- new net MOSI/1.5B: J1.14
- new net N$22: R4.2
- new net N$23: EPD_C8.2, J1.20
- new net N$25: C2-EP-DR1.1, D2.A, D4.K
- new net N$26: R_PWR_EPD.1
- new net N$27: EPD_C2.2, J1.4
- new net N$28: R1_EP_DR.1
- new net N$29: R_TYPE_SEL.2, SJ1.2
- new net N$31: EPD_C1.2, J1.5
- new net N$32: C32.2, IC2.REG
- new net N$34: J4.CC2, R2_USB.1
- new net N$37: J4.CC1, R1_USB.2
- new net N$39: EPD_C7.2, J1.19
- new net N$41: EPD_C6.2, J1.18
- new net N$42: EPD_C11.2, J1.23
- new net N$44: EPD_C12.2, J1.24
- new net OUT+: IC2.OUT+, TP_OP.TP
- new net OUT-: IC2.OUT-, TP_ON.TP
- new net P0.13/1.5D: C30.1, R5.1, SW_UP.2
- new net P0.14/1.5D: C31.1, R8.1, SW_ENT.2
- new net P1.01/1.6C: Q1.G
- new net P1.02/1.6C: C29.1, R7.1, SW_DN.2
- new net PREVGH: D5.K, EPD_C9.2, J1.21
- new net PREVGL: D4.A, EPD_C10.2, J1.22
- new net RESE: J1.3, Q3.S, R1_EP_DR.2
- new net SCK/1.5B: J1.13
- new net SCL/1.4C: IC2.SCL, U3.SCL
- new net SDA/1.4C: IC2.SDA, U3.SDA
- new net VBAT/1.2A: C27.1, TP_VBAT.TP, U3.CELL, U3.VDD
- new net VBUS/1.5D: C42.1, C43.1, D3.VBUS, J4.VBUS
- net 3V3/2.4A: now also J2.1; no longer J1.1
- net GND: now also C1-EP-DR.2, C27.2, C29.2, C30.2, C31.2, C32.1, C34.1, C42.2, C43.2, D2.K, D3.GND, EPD_C1.1, EPD_C10.1, EPD_C11.1, EPD_C12.1, EPD_C2.1, EPD_C5.1, EPD_C6.1, EPD_C7.1, EPD_C8.1, EPD_C9.1, IC2.GND, IC2.IN/TRIG, J1.17, J1.8, J1.MP1, J1.MP2, J2.3, J2.5, J4.GND, J4.SHIELD, R1_USB.1, R2_EP_DR.1, R2_USB.2, R9.1, R_TYPE_SEL.1, SJ1.1, SW_DN.1, SW_ENT.1, SW_UP.1, TP_BAT_GND.TP, U3.CTG, U3.EP, U3.GND, U3.QSTRT; no longer J1.3, J1.5
- net N$8: now also J2.6; no longer J1.6
- net SCL/2.4C: now also R4.1; no longer R2.1
- net SDA/2.4C: now also R2.1; no longer R1.1
- net SWDCLK: now also J2.4; no longer J1.4
- net SWDIO: now also J2.2; no longer J1.2
Other:
- note added: "Buttons"
- note added: "DMG2305UX-7"
- note added: "E-Paper Display Connector"
- note added: "E-Paper Drive Circuit"
- note added: "Fuel Gauge"
- note added: "Haptic Driver"
- note added: "USB C Connector & ESD Protection"
- moved on the sheet: C19, R2

Commit message: Made small changes to the schematic file and finished the .brd implementation.
Parts:
- ANT1: value 2450AT18B100E_2450AT18B100E -> 2450AT18B100E
- C1, C2: value (none) -> 12pF
- IC3: value BMA423_BMA423 -> BMA423
- IC9: value RT6160AWSC_RT6160AWSC -> RT6160AWSC
- L2: value 10µF -> 10µH
- U1: value NORDIC_NRF_4_NRF52840_QF -> NRF52840_QF
- renumbered C26 to C37, U$1 to U1
Connections:
- net GND1 renamed N$7
- removed net N$11: C9.1
- removed net N$20: R2.2
- removed net N$22: R4.2
- removed net N$26: R_PWR_EPD.1
- removed net N$28: R1_EP_DR.1
- removed net N$7 (its old number): U1.DEC5@N24
- removed net N$8: J2.6
- new net N$2: C9.1, U1.DEC5@N24
- net N$21: now also R2.2
- net N$29: now also R1_EP_DR.1
- net N$4: now also R4.2
- net P1.01/1.6C: now also R_PWR_EPD.1
- net RESET: now also J2.6
Other:
- moved on the sheet: ANT1, C1, C10, C11, C13, C2, C22, C3, C4, C9, L1

Commit message: Added files + README
Connections:
- removed net 3V3/1.7D: C34.2, IC2.VDD, Q1.S, R5.2, R7.2, R8.2, R_PWR_EPD.2
- removed net 3V3/2.4A: C12.1, C14.1, C19.1, C25.1, C33.1, C6.1, C7.1, C8.1, IC3.CSB, IC3.VDD, IC3.VDDIO, IC9.VOUT_1, IC9.VOUT_2, J2.1, R17.1, R18.1, TP5.TP, TP_3V3.TP, U1.VDD@A22, U1.VDD@AD14, U1.VDD@AD23, U1.VDD@B1, U1.VDD@W1, U1.VDDH@Y2
- removed net ALERT/1.6C: U3.!ALERT
- removed net ALERT/2.5C: U1.P0.10/NFC2@J24
- removed net D+/1.5D: D3.I/O2_2
- removed net D+/2.7D: U1.D+@AD6
- removed net D-/1.5D: D3.I/O1_2
- removed net D-/2.7D: U1.D-@AD4
- removed net EPD_BUSY/1.5D: J1.9
- removed net EPD_BUSY/2.2D: U1.P0.17@AD12
- removed net EPD_CS/1.4C: J1.12
- removed net EPD_CS/2.2D: U1.P0.05/AIN3@K2
- removed net EPD_DC/1.5D: J1.11
- removed net EPD_DC/2.2D: U1.P0.15@AD10
- removed net EPD_RST/1.5D: J1.10
- removed net EPD_RST/2.2D: U1.P0.16@AC11
- removed net HAPTIC_EN/1.4A: IC2.EN
- removed net HAPTIC_EN/2.6A: U1.P0.12@U1
- removed net MOSI/1.5B: J1.14
- removed net MOSI/2.2D: U1.P0.03/AIN1@B13
- removed net P0.13/1.5D: C30.1, R5.1, SW_UP.2
- removed net P0.13/2.6C: U1.P0.13@AD8
- removed net P0.14/1.5D: C31.1, R8.1, SW_ENT.2
- removed net P0.14/2.7C: U1.P0.14@AC9
- removed net P1.01/1.6C: Q1.G, R_PWR_EPD.1
- removed net P1.01/2.4B: U1.P1.01@Y23
- removed net P1.02/1.6C: C29.1, R7.1, SW_DN.2
- removed net P1.02/2.8C: U1.P1.02@W24
- removed net SCK/1.5B: J1.13
- removed net SCK/2.2D: U1.P0.02/AIN0@A12
- removed net SCL/1.4C: IC2.SCL, U3.SCL
- removed net SCL/2.4C: IC1.SCL, IC3.SCX, R17.2, R4.1, TP_SCL.TP, U1.P0.07@M2
- removed net SDA/1.4C: IC2.SDA, U3.SDA
- removed net SDA/2.4C: IC1.SDA, IC3.SDX, R18.2, R2.1, TP_SDA.TP, U1.P0.06@L1
- removed net VBAT/1.2A: C27.1, TP_VBAT.TP, U3.CELL, U3.VDD
- removed net VBAT/2.5C: C37.2, IC1.BAT
- removed net VBUS/1.5D: C42.1, C43.1, D3.VBUS, J4.VBUS
- removed net VBUS/2.6D: C21.1, C38.2, IC1.IN, U1.VBUS@AD2
- new net 3V3: C12.1, C14.1, C19.1, C25.1, C33.1, C34.2, C6.1, C7.1, C8.1, IC2.VDD, IC3.CSB, IC3.VDD, IC3.VDDIO, IC9.VOUT_1, IC9.VOUT_2, J2.1, Q1.S, R17.1, R18.1, R5.2, R7.2, R8.2, R_PWR_EPD.2, TP5.TP, TP_3V3.TP, U1.VDD@A22, U1.VDD@AD14, U1.VDD@AD23, U1.VDD@B1, U1.VDD@W1, U1.VDDH@Y2
- new net ALERT: U1.P0.10/NFC2@J24, U3.!ALERT
- new net D+: D3.I/O2_2, U1.D+@AD6
- new net D-: D3.I/O1_2, U1.D-@AD4
- new net EPD_BUSY: J1.9, U1.P0.17@AD12
- new net EPD_CS: J1.12, U1.P0.05/AIN3@K2
- new net EPD_DC: J1.11, U1.P0.15@AD10
- new net EPD_RST: J1.10, U1.P0.16@AC11
- new net HAPTIC_EN: IC2.EN, U1.P0.12@U1
- new net MOSI: J1.14, U1.P0.03/AIN1@B13
- new net P0.13: C30.1, R5.1, SW_UP.2, U1.P0.13@AD8
- new net P0.14: C31.1, R8.1, SW_ENT.2, U1.P0.14@AC9
- new net P1.01: Q1.G, R_PWR_EPD.1, U1.P1.01@Y23
- new net P1.02: C29.1, R7.1, SW_DN.2, U1.P1.02@W24
- new net SCK: J1.13, U1.P0.02/AIN0@A12
- new net SCL: IC1.SCL, IC2.SCL, IC3.SCX, R17.2, R4.1, TP_SCL.TP, U1.P0.07@M2, U3.SCL
- new net SDA: IC1.SDA, IC2.SDA, IC3.SDX, R18.2, R2.1, TP_SDA.TP, U1.P0.06@L1, U3.SDA
- new net VBAT: C27.1, C37.2, IC1.BAT, TP_VBAT.TP, U3.CELL, U3.VDD
- new net VBUS: C21.1, C38.2, C42.1, C43.1, D3.VBUS, IC1.IN, J4.VBUS, U1.VBUS@AD2
